File: kicad/io_board.kicad_sch (KiCad schematic)
At the start: 11 parts, among them J1 AudioJack2_SwitchT, J2 AudioJack2_SwitchT, U1 TL072

Commit message: Update KiCad project files and documentation
- Changed active layer in output_pcb.kicad_prl from 5 to 0.
- Updated project title, date, revision, and company in output_pcb.kicad_sch.
- Modified footprint properties for jacks in output_pcb.kicad_sch to use "Eurorack" library.
- Added README.md with project overview, features, quick start guide, file descriptions, build notes, testing procedures, and licensing information.
- Created a lock file for the schematic output.
Parts:
- J1, J2: footprint AudioJacks2:Jack_3.5mm_QingPu_WQP-PJ398SM_Vertical -> Eurorack:Jack_3.5mm_QingPu_WQP-PJ398SM_Vertical
- RV1, RV2: footprint AO_tht:Potentiometer_Alpha_RD902F-40-00D_Dual_Vertical_CircularHoles_centered -> Eurorack:Potentiometer_Alpha_RD902F-40-00D_Dual_Vertical_CircularHoles_centered
Changed lines of the file:
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@@
 			)
 		)
-		(property "Footprint" "AudioJacks2:Jack_3.5mm_QingPu_WQP-PJ398SM_Vertical"
+		(property "Footprint" "Eurorack:Jack_3.5mm_QingPu_WQP-PJ398SM_Vertical"
 			(at 36.83 99.06 0)
 			(effects
@@
 			)
 		)
-		(property "Footprint" "AO_tht:Potentiometer_Alpha_RD902F-40-00D_Dual_Vertical_CircularHoles_centered"
+		(property "Footprint" "Eurorack:Potentiometer_Alpha_RD902F-40-00D_Dual_Vertical_CircularHoles_centered"
 			(at 160.655 48.895 0)
 			(effects
@@
 			)
 		)
-		(property "Footprint" "AO_tht:Potentiometer_Alpha_RD902F-40-00D_Dual_Vertical_CircularHoles_centered"
+		(property "Footprint" "Eurorack:Potentiometer_Alpha_RD902F-40-00D_Dual_Vertical_CircularHoles_centered"
 			(at 128.905 48.895 0)
 			(effects
@@
 			)
 		)
-		(property "Footprint" "AudioJacks2:Jack_3.5mm_QingPu_WQP-PJ398SM_Vertical"
+		(property "Footprint" "Eurorack:Jack_3.5mm_QingPu_WQP-PJ398SM_Vertical"
 			(at 36.83 76.2 0)
 			(effects
