File: kicad/output_pcb.kicad_pcb (KiCad board)
At the start: 2 copper layers, 165 x 103.8 mm, 125 parts, among them J1 AudioJack2_SwitchT, J11 Conn_01x10_Pin, J12 Conn_01x10_Socket, J13 Conn_01x10_Pin, J2 AudioJack2_SwitchT, J21 Conn_01x10_Pin, J22 Conn_01x10_Socket, J23 Conn_01x10_Pin, J3 AudioJack3_SwitchTR, J4 AudioJack3_SwitchTR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

Commit message: Update KiCad project files and documentation
- Changed active layer in output_pcb.kicad_prl from 5 to 0.
- Updated project title, date, revision, and company in output_pcb.kicad_sch.
- Modified footprint properties for jacks in output_pcb.kicad_sch to use "Eurorack" library.
- Added README.md with project overview, features, quick start guide, file descriptions, build notes, testing procedures, and licensing information.
- Created a lock file for the schematic output.
Parts:
- J1, J2: footprint AudioJacks2:Jack_3.5mm_QingPu_WQP-PJ398SM_Vertical -> Eurorack:Jack_3.5mm_QingPu_WQP-PJ398SM_Vertical
- J3, J4, J5: footprint AO_tht:Jack_6.35mm_PJ_629HAN_slots -> Eurorack:Jack_6.35mm_PJ_629HAN_slots
- RV1, RV2: footprint AO_tht:Potentiometer_Alpha_RD902F-40-00D_Dual_Vertical_CircularHoles_centered -> Eurorack:Potentiometer_Alpha_RD902F-40-00D_Dual_Vertical_CircularHoles_centered
- moved D12 19.1 mm to (152.8, 132.0)
- moved D2 19.1 mm to (154.1, 53.3)
- moved D7 19.1 mm to (130.0, 132.0)
- moved R21 19.1 mm to (217.6, 50.1)
- moved R33 19.1 mm to (137.0, 66.0)
- moved R41 19.1 mm to (124.9, 104.7)
- moved R42 19.1 mm to (124.9, 118.0)
- moved C10 19.1 mm to (211.9, 131.4)
- moved C13 19.1 mm to (199.8, 106.7)
- moved C14 19.1 mm to (199.8, 114.9)
- moved C19 19.1 mm to (198.6, 57.6)
- moved C28 19.1 mm to (155.1, 69.2)
- moved C30 19.1 mm to (202.9, 140.9)
- moved C33 19.1 mm to (217.6, 45.0)
- moved C39 19.1 mm to (204.3, 111.0)
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