File: kicad/output_pcb.kicad_pcb (KiCad board)
At the start: 2 copper layers, 165 x 103.8 mm, 125 parts, among them J1 AudioJack2_SwitchT, J11 Conn_01x10_Pin, J12 Conn_01x10_Socket, J13 Conn_01x10_Pin, J2 AudioJack2_SwitchT, J21 Conn_01x10_Pin, J22 Conn_01x10_Socket, J23 Conn_01x10_Pin, J3 AudioJack3_SwitchTR, J4 AudioJack3_SwitchTR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

Commit message: change of text
Other:
- board text added: "designed in South Tyrol"
- board text removed: "made in South Tyrol"
Changed lines of the file:
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@@
 		(layer "Edge.Cuts")
 	)
-	(gr_text "made in\nSouth Tyrol"
-		(at 216.41 89.59 0)
+	(gr_text "designed in\nSouth Tyrol"
+		(at 215.485 89.805 0)
 		(layer "F.SilkS")
 		(effects
