File: kicad/output_pcb.kicad_sch (KiCad schematic)
At the start: 17 parts, among them J11 Conn_01x10_Pin, J12 Conn_01x10_Socket, J13 Conn_01x10_Pin, J21 Conn_01x10_Pin, J22 Conn_01x10_Socket, J23 Conn_01x10_Pin, J3 AudioJack3_SwitchTR, J4 AudioJack3_SwitchTR, J5 AudioJack3_SwitchTR, J6 Conn_02x05_Odd_Even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

Commit message: Update KiCad project files and documentation
- Changed active layer in output_pcb.kicad_prl from 5 to 0.
- Updated project title, date, revision, and company in output_pcb.kicad_sch.
- Modified footprint properties for jacks in output_pcb.kicad_sch to use "Eurorack" library.
- Added README.md with project overview, features, quick start guide, file descriptions, build notes, testing procedures, and licensing information.
- Created a lock file for the schematic output.
Parts:
- J3, J4, J5: footprint AO_tht:Jack_6.35mm_PJ_629HAN_slots -> Eurorack:Jack_6.35mm_PJ_629HAN_slots
Other:
- company: Free Modular -> Dirty Dream - Nathanael Noir
- title: Output -> Output Module with Volume Meter
Changed lines of the file:
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@@
 	(paper "A4")
 	(title_block
-		(title "Output")
-		(date "2024-03-18")
-		(rev "v1.1")
-		(company "Free Modular")
+		(title "Output Module with Volume Meter")
+		(date "2026-02-12")
+		(rev "v1.0")
+		(company "Dirty Dream - Nathanael Noir")
 	)
 	(junction
@@
 			)
 		)
-		(property "Footprint" "AO_tht:Jack_6.35mm_PJ_629HAN_slots"
+		(property "Footprint" "Eurorack:Jack_6.35mm_PJ_629HAN_slots"
 			(at 119.38 123.19 0)
 			(effects
@@
 			)
 		)
-		(property "Footprint" "AO_tht:Jack_6.35mm_PJ_629HAN_slots"
+		(property "Footprint" "Eurorack:Jack_6.35mm_PJ_629HAN_slots"
 			(at 125.73 35.56 0)
 			(effects
@@
 			)
 		)
-		(property "Footprint" "AO_tht:Jack_6.35mm_PJ_629HAN_slots"
+		(property "Footprint" "Eurorack:Jack_6.35mm_PJ_629HAN_slots"
 			(at 119.38 66.04 0)
 			(effects
